File: KiCAD Files/KiCAD Files.kicad_pcb (KiCad board)
At the start: 2 copper layers, 140 x 120 mm, 49 parts, among them J1 Power-Input, J10 SPI-Expansion, J11 I2C-Expansion, J12 Flow, J2 Pump-Conn, J3 Chopper-Conn, J4 Heater-Conn, J5 Term-1, J6 Term-2, J7 Humidity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

Commit message: Manually-Routed-V1
Parts:
- moved R10 10.1 mm to (180.2, 105.0), turned to 180 degrees
- moved R9 9.40 mm to (180.2, 101.0), turned to 180 degrees
- moved C3 0.99 mm to (138.0, 58.5)
Routing:
- net GND: track 0.00 -> 672.4 mm, vias 0 -> 7
- net +5V: track 0.00 -> 324.4 mm, vias 0 -> 6
- net VS: track 0.00 -> 191.2 mm
- net /Term-1: track 0.00 -> 139.1 mm, vias 0 -> 4
- net +12V: track 0.00 -> 135.1 mm, vias 0 -> 4
- net /Term-2: track 0.00 -> 119.5 mm, vias 0 -> 2
- net Net-(J10-Pin_2): track 0.00 -> 116.9 mm, vias 0 -> 2
- net +8V: track 0.00 -> 109.3 mm, vias 0 -> 2
- net Net-(D2-A): track 0.00 -> 88.4 mm
- net /Methane: track 0.00 -> 86.7 mm, vias 0 -> 2
- net +3.3V: track 0.00 -> 83.9 mm, vias 0 -> 2
- net /Flow: track 0.00 -> 72.6 mm, vias 0 -> 2
- net Net-(J10-Pin_3): track 0.00 -> 65.7 mm
- net /CO2: track 0.00 -> 64.3 mm, vias 0 -> 2
- net Net-(J10-Pin_4): track 0.00 -> 53.2 mm
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