File: KiCAD Files/KiCAD Files-Auto.kicad_pcb (KiCad board)
At the start: 2 copper layers, 140 x 120 mm, 49 parts, among them J1 Power-Input, J10 SPI-Expansion, J11 I2C-Expansion, J12 Flow, J2 Pump-Conn, J3 Chopper-Conn, J4 Heater-Conn, J5 Term-1, J6 Term-2, J7 Humidity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

Commit message: Finalized-2-Layer
Routing:
- net GND: track 672.4 -> 0.00 mm, vias 7 -> 0
- net +5V: track 324.4 -> 0.00 mm, vias 6 -> 0
- net VS: track 191.2 -> 0.00 mm
- net /Term-1: track 139.1 -> 0.00 mm, vias 4 -> 0
- net +12V: track 135.1 -> 0.00 mm, vias 4 -> 0
- net /Term-2: track 119.5 -> 0.00 mm, vias 2 -> 0
- net Net-(J10-Pin_2): track 116.9 -> 0.00 mm, vias 2 -> 0
- net +8V: track 109.3 -> 0.00 mm, vias 2 -> 0
- net Net-(D2-A): track 88.4 -> 0.00 mm
- net /Methane: track 86.7 -> 0.00 mm, vias 2 -> 0
- net +3.3V: track 83.9 -> 0.00 mm, vias 2 -> 0
- net /Flow: track 72.6 -> 0.00 mm, vias 2 -> 0
- net Net-(J10-Pin_3): track 65.7 -> 0.00 mm
- net /CO2: track 64.3 -> 0.00 mm, vias 2 -> 0
- net Net-(J10-Pin_4): track 53.2 -> 0.00 mm
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